Commit message: Fix small things

File: urdf/r2_robot.urdf (robot description, URDF)
Before this commit: robot flexible, 4 links, 3 joints
Links:
- link end: geometry visual box size=.15 .15 .1
Joints:
- joint link2_to_end: axis (none) -> 0 0 1; type fixed -> continuous

Commit message: Fix 2D problem and start fixing algorithm

File: urdf/r2_robot.urdf (robot description, URDF)
Before this commit: robot flexible, 4 links, 3 joints
Joints:
- joint base_to_link1: limit (none) -> lower=-3.15 upper=3.15 effort=15 velocity=5; type continuous -> revolute
- joint link1_to_link2: limit (none) -> lower=-3.15 upper=3.15 effort=15 velocity=5; type continuous -> revolute
- joint link2_to_end: limit (none) -> lower=-3.15 upper=3.15 effort=15 velocity=5; type continuous -> revolute

Commit message: Some fixes to pinnochio

File: urdf/r2_robot.urdf (robot description, URDF)
Before this commit: robot flexible, 4 links, 3 joints
Links:
- removed link base
- added link base_link; visual cylinder length=0.2 radius=0.1
Joints:
- joint base_to_link1: parent base -> base_link

Commit message: Fix jacobian

File: urdf/r2_robot.urdf (robot description, URDF)
Before this commit: robot flexible, 4 links, 3 joints
Links:
- removed link base_link
- added link base; visual cylinder length=0.2 radius=0.1
Joints:
- joint base_to_link1: parent base_link -> base
